File: FET_bord/FET_bord.brd (EAGLE design)
At the start: 85 x 54 mm, 70 parts

Commit message: 基板設計ほぼ終わりあとは仕上げ
Parts:
- moved U$13 44.5 mm to (14.0, 0.00)
- moved U$10 2.65 mm to (18.3, 20.4)
- moved U$9 2.65 mm to (41.1, 20.4)
- moved TR1 2.54 mm to (44.5, 30.5)
- moved TR3 2.54 mm to (21.6, 30.5)
- moved R16 1.80 mm to (14.0, 25.4)
- moved R11 1.27 mm to (34.3, 30.5)
- moved R12 1.27 mm to (11.4, 30.5)
- moved R15 1.27 mm to (38.1, 25.4)
- moved R17 1.27 mm to (14.0, 2.54)
- moved U$11 0.77 mm to (18.3, 13.7)
- moved U$12 0.77 mm to (41.1, 13.7)
Routing:
- net GLB: track 2.73 -> 69.2 mm, vias 0 -> 3
- net GHB: track 4.98 -> 46.1 mm
- net SB: track 12.1 -> 45.9 mm, vias 0 -> 35
- net VDD: track 96.0 -> 111.0 mm, vias 1 -> 2
- net N$28: track 9.70 -> 4.93 mm
- net N$27: track 9.70 -> 5.46 mm
- net GND: track 167.8 -> 164.0 mm
- net N$26: track 2.22 -> 5.46 mm
- net GLA: track 58.3 -> 59.3 mm
- net N$25: track 5.46 -> 4.93 mm
- net SA: vias 1 -> 35
- added copper zone on layer 1, net GND
- added copper zone on layer 16, net GND
- added copper zone on layer 1, net M
- added copper zone on layer 16, net M
- added copper zone on layer 1, net SA
- added copper zone on layer 16, net SA
- added copper zone on layer 1, net SB
- added copper zone on layer 16, net SB
- added copper zone on layer 1, net VDD
- added copper zone on layer 16, net VDD
