File: FET_bord/FET_bord.brd (EAGLE design)
At the start: 85 x 54 mm, 69 parts

Commit message: 基板エラー修正
Parts:
- moved R8 6.54 mm to (66.4, 12.6), flipped to the top, turned to 180 degrees
- moved C7 3.21 mm to (62.7, 12.6), flipped to the top, turned to 0 degrees
Connections:
- net V5: no longer R8.2
- net VDD: now also R8.2
Routing:
- net VDD: track 111.0 -> 121.9 mm
- net RESET: track 25.0 -> 30.4 mm, vias 3 -> 2
- net N$19: track 2.18 -> 4.06 mm, vias 1 -> 0
- net GNDI: track 27.6 -> 27.1 mm
- net N$20: track 2.28 -> 2.71 mm, vias 1 -> 0

Commit message: 集合抵抗value記入
Parts:
- R_I1, R_I2: value (none) -> 1k
Changed lines of the file:
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@@
 <attribute name="NAME" x="62.865" y="33.655" size="1.27" layer="26" rot="MR0"/>
 </element>
-<element name="R_I1" library="user_rcl" package="0603X4RESISTOR" value="" x="71.12" y="12.7" smashed="yes" rot="MR0">
+<element name="R_I1" library="user_rcl" package="0603X4RESISTOR" value="1k" x="71.12" y="12.7" smashed="yes" rot="MR0">
 <attribute name="NAME" x="73.0925" y="13.97" size="1.27" layer="26" rot="MR0"/>
 <attribute name="VALUE" x="73.0925" y="10.16" size="1.27" layer="28" rot="MR0"/>
 </element>
-<element name="R_I2" library="user_rcl" package="0603X4RESISTOR" value="" x="62.23" y="33.02" smashed="yes">
+<element name="R_I2" library="user_rcl" package="0603X4RESISTOR" value="1k" x="62.23" y="33.02" smashed="yes">
 <attribute name="NAME" x="60.1305" y="35.052" size="1.27" layer="25"/>
 <attribute name="VALUE" x="60.2575" y="30.48" size="1.27" layer="27"/>
