File: FET_bord/FET_bord.sch (EAGLE design)
At the start: 69 parts

Commit message: 基板エラー修正
Connections:
- net V5: no longer R8.2
- net VDD: now also R8.2
Changed lines of the file:
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@@
 <part name="GND13" library="supply1" library_urn="urn:adsk.eagle:library:371" deviceset="GND" device=""/>
 <part name="GND7" library="supply1" library_urn="urn:adsk.eagle:library:371" deviceset="GNDINT" device=""/>
+<part name="VDD5" library="supply1" library_urn="urn:adsk.eagle:library:371" deviceset="VDD" device=""/>
 </parts>
 <sheets>
@@
 <instance part="GND7" gate="G$1" x="-292.1" y="48.26" smashed="yes">
 <attribute name="VALUE" x="-294.64" y="45.72" size="1.778" layer="96"/>
+</instance>
+<instance part="VDD5" gate="G$1" x="15.24" y="91.44" smashed="yes">
+<attribute name="VALUE" x="12.7" y="88.9" size="1.778" layer="96" rot="R90"/>
 </instance>
 </instances>
@@
 <junction x="-38.1" y="25.4"/>
 </segment>
+<segment>
+<pinref part="VDD5" gate="G$1" pin="VDD"/>
+<pinref part="R8" gate="G$1" pin="2"/>
+<wire x1="15.24" y1="88.9" x2="15.24" y2="83.82" width="0.1524" layer="91"/>
+</segment>
 </net>
 <net name="M" class="0">
@@
 <wire x1="43.18" y1="76.2" x2="43.18" y2="78.74" width="0.1524" layer="91"/>
 <label x="43.18" y="78.74" size="1.778" layer="95"/>
-<pinref part="R8" gate="G$1" pin="2"/>
-<wire x1="15.24" y1="83.82" x2="35.56" y2="83.82" width="0.1524" layer="91"/>
-<wire x1="35.56" y1="83.82" x2="35.56" y2="76.2" width="0.1524" layer="91"/>
-<junction x="35.56" y="76.2"/>
-</segment>
-<segment>
+</segment>
+<segment>

Commit message: 集合抵抗value記入
Parts:
- R_I1, R_I2: value (none) -> 1k
Changed lines of the file:
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@@
 <part name="U$6" library="user_leds" deviceset="RGB_LED" device=""/>
 <part name="U$7" library="user_tr_fet_igbt" deviceset="FDC6305" device=""/>
-<part name="R_I1" library="user_rcl" deviceset="R_SHUGOU" device=""/>
-<part name="R_I2" library="user_rcl" deviceset="R_SHUGOU" device=""/>
+<part name="R_I1" library="user_rcl" deviceset="R_SHUGOU" device="" value="1k"/>
+<part name="R_I2" library="user_rcl" deviceset="R_SHUGOU" device="" value="1k"/>
 <part name="GNDI2" library="supply1" library_urn="urn:adsk.eagle:library:371" deviceset="GNDI" device=""/>
 <part name="VDD4" library="supply1" library_urn="urn:adsk.eagle:library:371" deviceset="VDD" device=""/>
