File: MCU_bord/MCU_bord.brd (EAGLE design)
At the start: 32 x 54 mm, 20 parts

Commit message: TIMピンの選択ミスったのなおした
Parts:
- moved U$4 28.2 mm to (1.27, 48.3)
- moved U$2 2.54 mm to (5.08, 33.0)
- moved C8 2.54 mm to (7.37, 35.7)
Connections:
- net A_CH: now also U$1.8; no longer U$1.20
- net B_CH: now also U$1.7; no longer U$1.19
- net COAST: now also U$1.28; no longer U$1.7
- net DIR: now also U$1.27; no longer U$1.6
- net FF1: now also U$1.6; no longer U$1.8
- net ID3: now also U$1.19; no longer U$1.27
- net ID4: now also U$1.20; no longer U$1.28
Routing:
- net DIR: track 44.7 -> 26.1 mm, vias 0 -> 2
- net COAST: track 42.3 -> 25.5 mm, vias 0 -> 2
- net +5V: track 49.9 -> 66.1 mm, vias 2 -> 4
- net ID4: track 26.9 -> 18.7 mm, vias 3 -> 1
- net ID3: track 24.7 -> 17.8 mm, vias 3 -> 1
- net FF1: track 39.6 -> 33.8 mm, vias 0 -> 2
- net +3V3: track 100.4 -> 96.6 mm
- net FF2: track 38.5 -> 34.8 mm
- net ID1: track 23.8 -> 23.1 mm
- net CAN_RX: track 12.3 -> 11.7 mm
- net A_CH: track 24.0 -> 24.5 mm
- net GND: track 69.0 -> 68.5 mm, vias 108 -> 135
- net B_CH: track 26.6 -> 26.9 mm, vias 1 -> 0
- net NRST: track 35.9 -> 35.6 mm, vias 6 -> 4
Other:
- board text added: "0.hayate MotaDora_MCU"

Commit message: ミス直し
Connections:
- net A_CH: now also U$1.7; no longer U$1.8
- net B_CH: now also U$1.6; no longer U$1.7
- net FF1: now also U$1.8; no longer U$1.6
Routing:
- net FF1: track 33.8 -> 33.2 mm
Changed lines of the file:
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@@
 <signal name="FF1">
 <contactref element="CON1" pad="P$2"/>
-<contactref element="U$1" pad="6"/>
-<wire x1="12.6209125" y1="29.192028125" x2="11.840940625" y2="29.972" width="0.1524" layer="1"/>
-<wire x1="11.840940625" y1="29.972" x2="11.303" y2="29.972" width="0.1524" layer="1"/>
-<via x="11.303" y="29.972" extent="1-16" drill="0.35"/>
-<via x="5.461" y="30.099" extent="1-16" drill="0.35"/>
-<wire x1="5.461" y1="30.099" x2="3.7338" y2="31.8262" width="0.1524" layer="1"/>
+<via x="6.731" y="28.829" extent="1-16" drill="0.35"/>
+<via x="4.699" y="30.734" extent="1-16" drill="0.35"/>
+<wire x1="4.699" y1="30.734" x2="3.7338" y2="31.6992" width="0.1524" layer="1"/>
 <wire x1="14.23" y1="48.46994375" x2="14.23" y2="51.3" width="0.1524" layer="1"/>
-<wire x1="11.303" y1="29.972" x2="11.176" y2="30.099" width="0.1524" layer="16"/>
-<wire x1="11.176" y1="30.099" x2="5.461" y2="30.099" width="0.1524" layer="16"/>
-<wire x1="3.7338" y1="31.8262" x2="3.7338" y2="37.97374375" width="0.1524" layer="1"/>
+<wire x1="6.604" y1="28.829" x2="6.731" y2="28.829" width="0.1524" layer="16"/>
+<wire x1="6.604" y1="28.829" x2="4.699" y2="30.734" width="0.1524" layer="16"/>
+<wire x1="3.7338" y1="31.6992" x2="3.7338" y2="37.97374375" width="0.1524" layer="1"/>
 <wire x1="3.7338" y1="37.97374375" x2="14.23" y2="48.46994375" width="0.1524" layer="1"/>
+<contactref element="U$1" pad="8"/>
+<wire x1="11.489540625" y1="28.060659375" x2="10.7212" y2="28.829" width="0.1524" layer="1"/>
+<wire x1="10.7212" y1="28.829" x2="6.731" y2="28.829" width="0.1524" layer="1"/>
 </signal>
 <signal name="COAST">
@@
 <signal name="B_CH">
 <contactref element="U$4" pad="PIN1"/>
-<contactref element="U$1" pad="7"/>
-<wire x1="12.055225" y1="28.62634375" x2="11.34456875" y2="29.337" width="0.1524" layer="1"/>
-<wire x1="4.03969375" y1="29.337" x2="2.54" y2="30.83669375" width="0.1524" layer="1"/>
+<wire x1="3.40469375" y1="29.972" x2="2.54" y2="30.83669375" width="0.1524" layer="1"/>
 <wire x1="1.9936875" y1="46.1176" x2="1.9124" y2="46.1176" width="0.1524" layer="1"/>
 <wire x1="1.9124" y1="46.1176" x2="1.27" y2="46.76" width="0.1524" layer="1"/>
 <wire x1="2.54" y1="45.5712875" x2="1.9936875" y2="46.1176" width="0.1524" layer="1"/>
-<wire x1="11.34456875" y1="29.337" x2="4.03969375" y2="29.337" width="0.1524" layer="1"/>
+<wire x1="11.72556875" y1="29.972" x2="11.43" y2="29.972" width="0.1524" layer="1"/>
+<wire x1="11.43" y1="29.972" x2="3.40469375" y2="29.972" width="0.1524" layer="1"/>
 <wire x1="2.54" y1="30.83669375" x2="2.54" y2="45.5712875" width="0.1524" layer="1"/>
+<contactref element="U$1" pad="6"/>
+<wire x1="11.72556875" y1="29.972" x2="11.840940625" y2="29.972" width="0.1524" layer="1"/>
+<wire x1="11.840940625" y1="29.972" x2="12.6209125" y2="29.192028125" width="0.1524" layer="1"/>
 </signal>
 <signal name="A_CH">
 <contactref element="U$4" pad="PIN3"/>
-<contactref element="U$1" pad="8"/>
-<wire x1="11.489540625" y1="28.060659375" x2="10.518" y2="29.0322" width="0.1524" layer="1"/>
-<wire x1="3.4798" y1="29.0322" x2="2.159" y2="30.353" width="0.1524" layer="1"/>
+<wire x1="2.159" y1="30.353" x2="3.0988" y2="29.4132" width="0.1524" layer="1"/>
 <via x="2.159" y="30.353" extent="1-16" drill="0.35"/>
 <wire x1="2.159" y1="30.353" x2="2.159" y2="43.561" width="0.1524" layer="16"/>
 <wire x1="2.159" y1="43.561" x2="1.96" y2="43.76" width="0.1524" layer="16"/>
 <wire x1="1.96" y1="43.76" x2="1.27" y2="43.76" width="0.1524" layer="16"/>
-<wire x1="10.518" y1="29.0322" x2="3.4798" y2="29.0322" width="0.1524" layer="1"/>
+<contactref element="U$1" pad="7"/>
+<wire x1="11.26836875" y1="29.4132" x2="12.055225" y2="28.62634375" width="0.1524" layer="1"/>
+<wire x1="3.0988" y1="29.4132" x2="11.26836875" y2="29.4132" width="0.1524" layer="1"/>
 </signal>
 <signal name="ID1">
