File: MCU_bord/MCU_bord.brd (EAGLE design)
At the start: 32 x 54 mm, 20 parts

Commit message: 基板エラー修正
Parts:
- removed R1: 10k, user_rcl:1608
- removed U$4: ZH_5P, user_conector:ZH_5P
- added CON3: (no value), user_conector:XH_5P
- moved R_I1 2.84 mm to (29.2, 14.0), turned to 0 degrees
- moved SW1 1.27 mm to (29.2, 12.7), turned to 180 degrees
Connections:
- removed net N$7: IC1.P$8, R1.2
- net +3V3: now also SW1.P$5, SW1.P$6, SW1.P$7, SW1.P$8; no longer R_I1.5, R_I1.6, R_I1.7, R_I1.8
- net +5V: now also CON3.P$2; no longer R1.1, U$4.PIN2
- net A_CH: now also CON3.P$3; no longer U$4.PIN3
- net B_CH: now also CON3.P$1; no longer U$4.PIN1
- net GND: now also CON3.P$5, IC1.P$8, R_I1.1, R_I1.2, R_I1.3, R_I1.4; no longer SW1.P$1, SW1.P$2, SW1.P$3, SW1.P$4, U$4.PIN5
- net ID1: now also R_I1.8, SW1.P$1; no longer R_I1.1, SW1.P$8
- net ID2: now also R_I1.7, SW1.P$2; no longer R_I1.2, SW1.P$7
- net ID3: now also R_I1.6, SW1.P$3; no longer R_I1.3, SW1.P$6
- net ID4: now also R_I1.5, SW1.P$4; no longer R_I1.4, SW1.P$5
Routing:
- net ID1: track 23.1 -> 27.5 mm
- net ID2: track 16.9 -> 21.2 mm
- net +5V: track 66.1 -> 61.9 mm, vias 4 -> 3
- net ID4: track 18.7 -> 15.1 mm
- net N$7: track 2.79 -> 0.00 mm, vias 1 -> 0
- net B_CH: track 27.3 -> 29.5 mm
- net A_CH: track 24.8 -> 25.7 mm, vias 1 -> 0
- net ID3: track 17.8 -> 18.4 mm
- net +3V3: track 96.6 -> 96.0 mm
- net GND: track 68.5 -> 68.8 mm, vias 135 -> 131

Commit message: canトランシーバ終端抵抗追加、電源確認用LED追加
Parts:
- added LED1: (no value), user_leds:1608
- added R1: 120, user_rcl:1608
- added R3: 1k, user_rcl:1608
Connections:
- new net N$4: LED1.A, R3.2
- net +3V3: now also R3.1
- net CAN_N: now also R1.1
- net CAN_P: now also R1.2
- net GND: now also LED1.K
Routing:
- net +3V3: track 96.0 -> 100.0 mm
- net N$4: track 0.00 -> 3.07 mm
- net CAN_P: track 10.7 -> 11.0 mm, vias 0 -> 1
- net CAN_N: track 13.0 -> 13.3 mm, vias 1 -> 2
- net GND: vias 131 -> 130
Changed lines of the file:
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@@
 <element name="R_I1" library="user_rcl" package="1005X4RESISTOR" value="" x="29.21" y="13.97" smashed="yes" rot="MR0"/>
 <element name="CON3" library="user_conector" package="XH_5P" value="" x="0" y="50.8" smashed="yes" rot="R270"/>
+<element name="R1" library="user_rcl" package="1608" value="120" x="20.32" y="10.16" smashed="yes" rot="MR180">
+<attribute name="NAME" x="19.685" y="9.525" size="1.27" layer="26" rot="MR180"/>
+<attribute name="VALUE" x="19.685" y="12.065" size="1.27" layer="28" rot="MR180"/>
+</element>
+<element name="LED1" library="user_leds" package="1608" value="" x="13.97" y="41.91" smashed="yes" rot="R90">
+<attribute name="NAME" x="12.7" y="40.64" size="0.4064" layer="25" rot="R90"/>
+<attribute name="VALUE" x="13.208" y="40.64" size="0.4064" layer="27" rot="R90"/>
+</element>
+<element name="R3" library="user_rcl" package="1608" value="1k" x="16.51" y="43.18" smashed="yes" rot="R270">
+<attribute name="NAME" x="17.145" y="43.815" size="1.27" layer="25" rot="R270"/>
+<attribute name="VALUE" x="14.605" y="43.815" size="1.27" layer="27" rot="R270"/>
+</element>
 </elements>
 <signals>
@@
 <wire x1="26.73" y1="4.60815625" x2="25.4665625" y2="5.87159375" width="0.1524" layer="1"/>
 <wire x1="26.73" y1="3.3" x2="26.73" y2="4.60815625" width="0.1524" layer="1"/>
+<contactref element="R1" pad="2"/>
+<wire x1="21.17" y1="10.16" x2="21.01" y2="10" width="0.254" layer="16"/>
+<wire x1="21.01" y1="10" x2="20.955" y2="10" width="0.254" layer="16"/>
+<via x="20.955" y="10" extent="1-16" drill="0.35"/>
 </signal>
 <signal name="CAN_N">
@@
 <wire x1="23.48900625" y1="5.08" x2="19.685" y2="8.88400625" width="0.1524" layer="1"/>
 <wire x1="25.4" y1="5.08" x2="23.48900625" y2="5.08" width="0.1524" layer="1"/>
+<contactref element="R1" pad="1"/>
+<wire x1="19.47" y1="10.16" x2="19.525" y2="10.16" width="0.254" layer="16"/>
+<wire x1="19.525" y1="10.16" x2="19.685" y2="10" width="0.254" layer="16"/>
+<via x="19.685" y="10" extent="1-16" drill="0.35"/>
 </signal>
 <signal name="GND">
@@
 <via x="11.43" y="39.37" extent="1-16" drill="0.35"/>
 <via x="12.7" y="40.64" extent="1-16" drill="0.35"/>
-<via x="13.97" y="41.91" extent="1-16" drill="0.35"/>
 <via x="15.24" y="43.18" extent="1-16" drill="0.35"/>
 <via x="16.51" y="40.64" extent="1-16" drill="0.35"/>
@@
 <contactref element="R_I1" pad="1"/>
 <contactref element="CON3" pad="P$5"/>
+<contactref element="LED1" pad="K"/>
 </signal>
 <signal name="+5V">
@@
 <wire x1="22.86" y1="11.43" x2="19.05" y2="11.43" width="0.1524" layer="1"/>
 <wire x1="25.38" y1="8.91" x2="22.86" y2="11.43" width="0.1524" layer="1"/>
+<contactref element="R3" pad="1"/>
+<wire x1="16.51" y1="44.03" x2="16.93" y2="44.03" width="0.254" layer="1"/>
+<wire x1="18.923" y1="42.037" x2="18.923" y2="41.275" width="0.254" layer="1"/>
+<wire x1="16.93" y1="44.03" x2="18.923" y2="42.037" width="0.254" layer="1"/>
 </signal>
 <signal name="CAN_TX">
@@
 <wire x1="26.67" y1="20.32" x2="26.67" y2="16.51" width="0.1524" layer="1"/>
 </signal>
+<signal name="N$4">
+<contactref element="R3" pad="2"/>
+<contactref element="LED1" pad="A"/>
+<wire x1="13.97" y1="41.06" x2="15.24" y2="41.06" width="0.254" layer="1"/>
+<wire x1="15.24" y1="41.06" x2="16.51" y2="42.33" width="0.254" layer="1"/>
+</signal>
 </signals>
